File: Design/Rpi_schematics.sch (KiCad schematic (older format))
At the start: 10 parts

Commit message: more changes
Parts:
- removed P?: Ultrasonic Door, symbol CONN_4
- removed R1: 4.7k, ~, symbol R
- removed R10: 10, ~, symbol R
- added C?: 1u, ~, symbol CP1
- added K?: PIR, symbol CONN_3
- added LDR: 0, ~, symbol R
- added R? (x2): 1k, ~, symbol R
- added R?: 2.2k, ~, symbol R
- added SW? (x2): SW_PUSH, ~, symbol SW_PUSH
- P?: value TV Proximity Sensor -> SR04
Connections:
- net labels added: Relay1, Relay2, Relay3, Relay4
- net labels removed: Coffermaker, Door Bell LED
- wire segments 41 -> 59
- no-connect marks 0 -> 5
Other:
- moved on the sheet: K?, P?, R?
